Commit message: update urdf

File: turtlebot3_manipulation_description/urdf/open_manipulator_x.urdf.xacro (robot description, xacro)
@@ -156,27 +156,4 @@
     </inertial>
   </link>
-  <!--  Gripper link -->
-  <link name="gripper_link">
-    <visual>
-      <origin xyz="0.0 0.0 0" rpy="0 0 0"/>
-      <geometry>
-        <mesh filename="package://turtlebot3_manipulation_description/meshes/chain_link_grip_l.stl" scale="0.001 0.001 0.001"/>
-      </geometry>
-      <material name="grey"/>
-    </visual>
-    <collision>
-      <origin xyz="0.0 0.0 0" rpy="0 0 0"/>
-      <geometry>
-        <mesh filename="package://turtlebot3_manipulation_description/meshes/chain_link_grip_l.stl" scale="0.001 0.001 0.001"/>
-      </geometry>
-    </collision>
-    <inertial>
-      <origin xyz="0 0 0" />
-      <mass value="1.0e-03" />
-      <inertia ixx="1.0e-03" ixy="0.0" ixz="0.0"
-               iyy="1.0e-03" iyz="0.0"
-               izz="1.0e-03" />
-    </inertial>
-  </link>
   <!--  Gripper joint -->
   <joint name="gripper" type="prismatic">
@@ -187,17 +164,17 @@
     <limit velocity="4.8" effort="1" lower="-0.010" upper="0.019" />
   </joint>
-  <!--  Gripper link sub -->
-  <link name="gripper_link_sub">
-    <visual>
-      <origin xyz="0.0 -0.0 0" rpy="0 0 0"/>
-      <geometry>
-        <mesh filename="package://turtlebot3_manipulation_description/meshes/chain_link_grip_r.stl" scale="0.001 0.001 0.001"/>
-      </geometry>
-      <material name="grey"/>
-    </visual>
-    <collision>
-      <origin xyz="0.0 -0.0 0" rpy="0 0 0"/>
-      <geometry>
-        <mesh filename="package://turtlebot3_manipulation_description/meshes/chain_link_grip_r.stl" scale="0.001 0.001 0.001"/>
+  <!--  Gripper link -->
+  <link name="gripper_link">
+    <visual>
+      <origin xyz="0.0 0.0 0" rpy="0 0 0"/>
+      <geometry>
+        <mesh filename="package://turtlebot3_manipulation_description/meshes/chain_link_grip_l.stl" scale="0.001 0.001 0.001"/>
+      </geometry>
+      <material name="grey"/>
+    </visual>
+    <collision>
+      <origin xyz="0.0 0.0 0" rpy="0 0 0"/>
+      <geometry>
+        <mesh filename="package://turtlebot3_manipulation_description/meshes/chain_link_grip_l.stl" scale="0.001 0.001 0.001"/>
       </geometry>
     </collision>
@@ -219,4 +196,27 @@
     <mimic joint="gripper" multiplier="1"/>
   </joint>
+  <!--  Gripper link sub -->
+  <link name="gripper_link_sub">
+    <visual>
+      <origin xyz="0.0 -0.0 0" rpy="0 0 0"/>
+      <geometry>
+        <mesh filename="package://turtlebot3_manipulation_description/meshes/chain_link_grip_r.stl" scale="0.001 0.001 0.001"/>
+      </geometry>
+      <material name="grey"/>
+    </visual>
+    <collision>
+      <origin xyz="0.0 -0.0 0" rpy="0 0 0"/>
+      <geometry>
+        <mesh filename="package://turtlebot3_manipulation_description/meshes/chain_link_grip_r.stl" scale="0.001 0.001 0.001"/>
+      </geometry>
+    </collision>
+    <inertial>
+      <origin xyz="0 0 0" />
+      <mass value="1.0e-03" />
+      <inertia ixx="1.0e-03" ixy="0.0" ixz="0.0"
+               iyy="1.0e-03" iyz="0.0"
+               izz="1.0e-03" />
+    </inertial>
+  </link>
   <!-- end effector joint -->
   <joint name="end_effector_joint" type="fixed">
